File: Hardware/Wimos-Accelerometro/WIMOS-Accelerometro.sch (EAGLE design)
At the start: 9 parts, among them IC1 LD117AS33TR

Commit message: DOC + HW
Doc incremento 1 y 2 (Implementación)
Other:
- moved on the sheet: C1, C2, IC1, JP1, R1, R2, R3
