File: Hardware/Wimos-Central/WIMOS-motherboard.sch (EAGLE design)
At the start: 15 parts, among them IC2 LD117AS12TR, T1 2N2222, T2 2N2222

Commit message: DOC + HW
Doc incremento 1 y 2 (Implementación)
Parts:
- removed D1: 1N4148DO35-7, diode:1N4148DO35-7
- removed R2, R3, R4, R5, R6: (no value), rcl:R-EU_0204/5
- removed T1, T2: 2N2222, transistor-neu-to92:2N2222
- added R10, R7, R8: 2.2k, rcl:R-EU_0204/5
- added R9: 1k, rcl:R-EU_0204/5
- added T3: KSP2222A, transistor:MPS2222A-NPN-TO92-CBE
- R1: value (none) -> 2.2k
Connections:
- removed net N$2: D1.C, R3.2, T2.B
- removed net N$3: R4.1, R5.1, T1.B
- new net 3V3: U$1.3V
- new net N$4: R8.2, T3.B
- net 3.3V: now also R8.1; no longer R6.1
- net GND: now also R10.2; no longer D1.A, R5.2, T1.E, T2.E
- net RX_5V: now also R7.2, T3.C, U$1.D8; no longer R2.1, T2.C, U$1.D9
- net TX_5V: now also R9.1, U$1.D9; no longer R4.2, U$1.D8
- net VCC: now also R7.1; no longer R2.2
- net XBEE_RX: now also R10.1, R9.2; no longer R6.2, T1.C
- net XBEE_TX: now also T3.E; no longer R3.1
Other:
- note added: "n2.IM01"
- note added: "n2.IM02"
- note added: "n2.IM03"
- note added: "n2.IM04"
- note added: "n2.IM05"
- moved on the sheet: C1, C2, IC2, LED1, R1, ZIGBEE_MODULE
