File: Hardware/Wimos-Estación/WIMOS-motherboard.sch (EAGLE design)
At the start: 38 parts, among them IC1 7805T

Commit message: DOC + HW
Doc incremento 1 y 2 (Implementación)
Other:
- note added: "Connect to digital pinout."
- note added: "LED de estado"
- note added: "Lector de batería"
- note added: "n1.IM01"
- note added: "n1.IM02"
- note added: "n1.IM03"
- note added: "n1.IM04"
- note added: "n1.IM05"
- note added: "n1.IM06"
- note added: "n1.IM07"
- note added: "n1.IM08"
- note added: "n1.IM09"
- note added: "n1.IM10"
- note added: "n1.IM11"
- note added: "n1.IM12"
- note removed: "Estado de Bateria"
- note removed: "LED ON"
- moved on the sheet: A5, D3, D4, D5, LED2, R1, R17, R18
